File: Hardware_REG1_Front/REG1-Front-Dali.kicad_pcb (KiCad board)
At the start: 2 copper layers, 25.4 x 52.8 mm, 12 parts, among them J1 Conn_02x04_Odd_Even, SW1 Prog, SW2 Func, SW3 Res, SW4 BL

Commit message: updated front
Other:
- board text added: "GW-Dali"
- board text added: "REG1-Front-Dali V00.01 © thewhobox, 2023"
- board text removed: "REG1-Front-Universal V00.02 © Ing-Dom, 2022"
Changed lines of the file:
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@@
     (effects (font (size 1 1) (thickness 0.15)) (justify mirror))
   )
-  (gr_text "REG1-Front-Universal\nV00.02 © Ing-Dom, 2022" (at 111.59 130.94 90) (layer "B.SilkS")
+  (gr_text "REG1-Front-Dali\nV00.01 © thewhobox, 2023" (at 111.59 130.546 90) (layer "B.SilkS")
     (effects (font (size 1 1) (thickness 0.15)) (justify left mirror))
   )
@@
     (effects (font (size 1.5 1.5) (thickness 0.2)) (justify left))
   )
+  (gr_text "GW-Dali" (at 99.934 114.036) (layer "F.SilkS")
+    (effects (font (size 2 2) (thickness 0.3) bold) (justify left bottom))
+  )
   (gr_text "Reset" (at 103.75 131.75) (layer "F.SilkS")
