File: Hardware_REG1_App/REG1-App-Dali.kicad_sch (KiCad schematic)
At the start: 26 parts, among them J1 REG1_App_Connector, J2 Dali, Q1 BSS123, Q2 BC857, U1 EL817S1(C)(TU)-F, U2 EL817S1(C)(TU)-F, U3 STN93003, U4 STN1HNK60

Commit message: adapted to REG1-V1 and JLCPCB fabrication toolkit
Parts:
- BR1: footprint SOP245P670X290-4N -> DALI:SOP245P670X290-4N; LCSC (none) -> C2488
- C1: LCSC (none) -> C1588
- C2: LCSC (none) -> C49217
- D1: footprint DIOM4325X250N -> DALI:DIOM4325X250N; LCSC (none) -> C260228
- D2: LCSC (none) -> C111753
- D3: footprint SODFL2512X90N -> DALI:SODFL2512X90N; LCSC (none) -> C122985
- D4: LCSC (none) -> C2290
- J1: LCSC (none) -> C492418
- J2: LCSC (none) -> C441173
- Q1: footprint DALI:SOT23 -> Package_TO_SOT_SMD:SOT-23; JLCPCB Rotation Offset (none) -> 180; LCSC (none) -> C431506
- Q2: JLCPCB Rotation Offset (none) -> 180; LCSC (none) -> C8666
- R1, R2, R4, R5: LCSC (none) -> C17900
- R10: LCSC (none) -> C4410
- R11: LCSC (none) -> C17887
- R3: LCSC (none) -> C23151
- R6: LCSC (none) -> C17490
- R7, R8, R9: LCSC (none) -> C23162
- U1, U2: LCSC (none) -> C106900
- U3: footprint SOT230P700X180-4N -> DALI:SOT230P700X180-4N; JLCPCB Rotation Offset (none) -> -90; LCSC (none) -> C880083
- U4: JLCPCB Rotation Offset (none) -> -90; LCSC (none) -> C39303
Other:
- title: REG1-App-Universal -> REG1-App-Dali
Changed lines of the file:
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@@
   (paper "A4")
   (title_block
-    (title "REG1-App-Universal")
-    (date "2023-01-31")
-    (rev "V00.10")
+    (title "REG1-App-Dali")
+    (date "2023-11-07")
+    (rev "V00.90")
     (company "OpenKNX")
-    (comment 1 "by Ing-Dom <dom@ing-dom.de>")
+    (comment 1 "by thewhobox")
     (comment 4 "https://OpenKNX.de")
   )
@@
     )
     (property "Datasheet" "" (at 68.58 179.07 0)
+      (effects (font (size 1.27 1.27)) hide)
+    )
+    (property "LCSC" "C492418" (at 68.58 179.07 0)
       (effects (font (size 1.27 1.27)) hide)
     )
@@
       (effects (font (size 1.27 1.27)) hide)
     )
+    (property "LCSC" "C23151" (at 115.57 62.23 0)
+      (effects (font (size 1.27 1.27)) hide)
+    )
     (pin "1")
     (pin "2")
@@
       (effects (font (size 1.27 1.27)) hide)
     )
+    (property "LCSC" "C49217" (at 170.18 120.65 0)
+      (effects (font (size 1.27 1.27)) hide)
+    )
     (pin "1")
     (pin "2")
@@
       (effects (font (size 1.27 1.27)) hide)
     )
+    (property "LCSC" "C17490" (at 97.79 130.81 0)
+      (effects (font (size 1.27 1.27)) hide)
+    )
     (pin "1")
     (pin "2")
@@
     )
     (property "Datasheet" "~" (at 78.74 102.87 0)
+      (effects (font (size 1.27 1.27)) hide)
+    )
+    (property "LCSC" "C17900" (at 78.74 102.87 0)
       (effects (font (size 1.27 1.27)) hide)
     )
@@
       (effects (font (size 1.27 1.27)) (justify left) hide)
     )
+    (property "LCSC" "C8666" (at 102.87 44.45 0)
+      (effects (font (size 1.27 1.27)) hide)
+    )
+    (property "JLCPCB Rotation Offset" "180" (at 102.87 44.45 0)
+      (effects (font (size 1.27 1.27)) hide)
+    )
     (pin "1")
     (pin "2")
@@
       (effects (font (size 1.27 1.27)) hide)
     )
+    (property "LCSC" "C4410" (at 241.3 58.42 0)
+      (effects (font (size 1.27 1.27)) hide)
+    )
     (pin "1")
     (pin "2")
@@
       (effects (font (size 1.27 1.27)) hide)
     )
+    (property "LCSC" "C23162" (at 252.73 17.78 0)
+      (effects (font (size 1.27 1.27)) hide)
+    )
     (pin "1")
     (pin "2")
@@
     )
     (property "Datasheet" "~" (at 257.81 25.4 0)
+      (effects (font (size 1.27 1.27)) hide)
+    )
+    (property "LCSC" "C2290" (at 257.81 25.4 0)
       (effects (font (size 1.27 1.27)) hide)
     )
@@
       (effects (font (size 1.27 1.27)) hide)
     )
+    (property "LCSC" "C441173" (at 22.86 85.09 0)
+      (effects (font (size 1.27 1.27)) hide)
+    )
     (pin "1")
     (pin "2")
@@
       (effects (font (size 1.27 1.27)) (justify bottom) hide)
     )
+    (property "LCSC" "C39303" (at 111.76 105.41 0)
+      (effects (font (size 1.27 1.27)) hide)
+    )
+    (property "JLCPCB Rotation Offset" "-90" (at 111.76 105.41 0)
+      (effects (font (size 1.27 1.27)) hide)
+    )
     (pin "1")
     (pin "2")
@@
     )
     (property "Datasheet" "~" (at 242.57 25.4 0)
+      (effects (font (size 1.27 1.27)) hide)
+    )
+    (property "LCSC" "C23162" (at 242.57 25.4 0)
       (effects (font (size 1.27 1.27)) hide)
     )
@@
       (effects (font (size 1.27 1.27)) (justify bottom) hide)
     )
+    (property "LCSC" "C106900" (at 215.9 60.96 0)
+      (effects (font (size 1.27 1.27)) hide)
+    )
     (pin "1")
     (pin "2")
@@
     )
     (property "Datasheet" "~" (at 78.74 92.71 0)
+      (effects (font (size 1.27 1.27)) hide)
+    )
+    (property "LCSC" "C17900" (at 78.74 92.71 0)
       (effects (font (size 1.27 1.27)) hide)
     )
@@
       (effects (font (size 1.27 1.27)) (justify left))
     )
-    (property "Footprint" "SOT230P700X180-4N" (at 113.03 34.29 0)
+    (property "Footprint" "DALI:SOT230P700X180-4N" (at 113.03 34.29 0)
       (effects (font (size 1.27 1.27)) (justify bottom) hide)
     )
     (property "Datasheet" "" (at 113.03 34.29 0)
+      (effects (font (size 1.27 1.27)) hide)
+    )
+    (property "LCSC" "C880083" (at 113.03 34.29 0)
+      (effects (font (size 1.27 1.27)) hide)
+    )
+    (property "JLCPCB Rotation Offset" "-90" (at 113.03 34.29 0)
       (effects (font (size 1.27 1.27)) hide)
     )
@@
       (effects (font (size 1.27 1.27)) (justify right))
     )
-    (property "Footprint" "SODFL2512X90N" (at 181.61 120.65 0)
+    (property "Footprint" "DALI:SODFL2512X90N" (at 181.61 120.65 0)
       (effects (font (size 1.27 1.27)) (justify bottom) hide)
     )
@@
     (property "MANUFACTURER" "Rohm Semiconductor" (at 181.61 120.65 0)
       (effects (font (size 1.27 1.27)) (justify bottom) hide)
+    )
+    (property "LCSC" "C122985" (at 181.61 120.65 0)
+      (effects (font (size 1.27 1.27)) hide)
     )
     (pin "A")
@@
       (effects (font (size 1.27 1.27)))
     )
-    (property "Footprint" "SOP245P670X290-4N" (at 39.37 174.93 0)
+    (property "Footprint" "DALI:SOP245P670X290-4N" (at 39.37 174.93 0)
       (effects (font (size 1.27 1.27)) (justify left top) hide)
     )
@@
       (effects (font (size 1.27 1.27)) (justify left top) hide)
     )
+    (property "LCSC" "C2488" (at 58.42 80.01 0)
+      (effects (font (size 1.27 1.27)) hide)
+    )
     (pin "1")
     (pin "2")
@@
       (effects (font (size 1.27 1.27)) hide)
     )
+    (property "LCSC" "C1588" (at 152.4 120.65 0)
+      (effects (font (size 1.27 1.27)) hide)
+    )
     (pin "1")
     (pin "2")
@@
       (effects (font (size 1.27 1.27)) hide)
     )
+    (property "LCSC" "C23162" (at 137.16 120.65 0)
+      (effects (font (size 1.27 1.27)) hide)
+    )
     (pin "1")
     (pin "2")
@@
     (property "AVAILABILITY" "Good" (at 215.9 27.94 0)
       (effects (font (size 1.27 1.27)) (justify bottom) hide)
+    )
+    (property "LCSC" "C106900" (at 215.9 27.94 0)
+      (effects (font (size 1.27 1.27)) hide)
     )
     (pin "1")
@@
       (effects (font (size 1.27 1.27)) hide)
     )
+    (property "LCSC" "C17900" (at 90.17 34.29 0)
+      (effects (font (size 1.27 1.27)) hide)
+    )
     (pin "1")
     (pin "2")
@@
       (effects (font (size 1.27 1.27)) hide)
     )
+    (property "LCSC" "C17887" (at 252.73 58.42 0)
+      (effects (font (size 1.27 1.27)) hide)
+    )
     (pin "1")
     (pin "2")
@@
       (effects (font (size 1.27 1.27)) (justify left))
     )
-    (property "Footprint" "DALI:SOT23" (at 123.19 120.65 0)
+    (property "Footprint" "Package_TO_SOT_SMD:SOT-23" (at 123.19 120.65 0)
       (effects (font (size 1.27 1.27)) (justify bottom) hide)
     )
@@
       (effects (font (size 1.27 1.27)) hide)
     )
+    (property "LCSC" "C431506" (at 123.19 120.65 0)
+      (effects (font (size 1.27 1.27)) hide)
+    )
+    (property "JLCPCB Rotation Offset" "180" (at 123.19 120.65 0)
+      (effects (font (size 1.27 1.27)) hide)
+    )
     (pin "1")
     (pin "2")
@@
       (effects (font (size 1.27 1.27)) hide)
     )
+    (property "LCSC" "C17900" (at 77.47 34.29 0)
+      (effects (font (size 1.27 1.27)) hide)
+    )
     (pin "1")
     (pin "2")
@@
       (effects (font (size 1.27 1.27)) hide)
     )
+    (property "LCSC" "C111753" (at 78.74 113.03 0)
+      (effects (font (size 1.27 1.27)) hide)
+    )
     (pin "1")
     (pin "2")
@@
       (effects (font (size 1.27 1.27)) (justify right))
     )
-    (property "Footprint" "DIOM4325X250N" (at 78.74 132.08 0)
+    (property "Footprint" "DALI:DIOM4325X250N" (at 78.74 132.08 0)
       (effects (font (size 1.27 1.27)) (justify bottom) hide)
     )
@@
       (effects (font (size 1.27 1.27)) (justify bottom) hide)
     )
+    (property "LCSC" "C260228" (at 78.74 132.08 0)
+      (effects (font (size 1.27 1.27)) hide)
+    )
     (pin "A")
